Commit message: remove grid

File: models/rm2/rm2.urdf (robot description, URDF)
Before this commit: robot rm2_sim, 4 links, 3 joints
Links:
- removed link b::bLink
- added link base_link
- added link d_435_camera
- added link l1::fLink
- added link l1::mLink
- added link l2::fLink
- added link l2::mLink
- added link l3::fLink
- added link l3::mLink
- added link sa1::aLink
- added link sa1::ccwaLink
- added link sa1::cwaLink
- added link sa1::sbLink
- added link sa2::aLink
- added link sa2::ccwaLink
- added link sa2::cwaLink
- added link sa2::sbLink
- added link sa3::aLink
- added link sa3::ccwaLink
- added link sa3::cwaLink
- added link sa3::sbLink
- added link wa2::aLink
- added link wa2::fwLink
- added link wa2::rwLink
- added link wa2::wbLink
- added link wa3::aLink
- added link wa3::fwLink
- added link wa3::rwLink
- added link wa3::wbLink
Joints:
- added joint j_l1_sa1: type fixed, parent l1::fLink, child sa1::aLink, origin xyz=0.0035 0.024 0.0473 rpy=0 0 0
- added joint j_l2_sa2: type fixed, parent l2::fLink, child sa2::aLink, origin xyz=0.0035 0.024 0.0473 rpy=0 0 0
- added joint j_l2_wa2: type fixed, parent l2::fLink, child wa2::aLink, origin xyz=0.0035 0.024 0.0473 rpy=0 0 0
- added joint j_l3_sa3: type fixed, parent l3::fLink, child sa3::aLink, origin xyz=0.0035 0.024 0.0473 rpy=0 0 0
- added joint j_l3_wa3: type fixed, parent l3::fLink, child wa3::aLink, origin xyz=0.0035 0.024 0.0473 rpy=0 0 0
- added joint j_rgbd_b: type fixed, parent base_link, child d_435_camera, origin xyz=0.090 0 0.038911 rpy=0 0 0
- added joint l1::j_l_m: type fixed, parent l1::lLink, child l1::mLink
- added joint l1::j_m_f: type fixed, parent l1::mLink, child l1::fLink
- added joint l2::j_l_m: type fixed, parent l2::lLink, child l2::mLink
- added joint l2::j_m_f: type fixed, parent l2::mLink, child l2::fLink
- added joint l3::j_l_m: type fixed, parent l3::lLink, child l3::mLink
- added joint l3::j_m_f: type fixed, parent l3::mLink, child l3::fLink
- added joint sa1::j_a_sb: type fixed, parent sa1::aLink, child sa1::sbLink
- added joint sa1::j_sb_ccwa: type continuous, parent sa1::sbLink, child sa1::ccwaLink, axis 0 0 1
- added joint sa1::j_sb_cwa: type continuous, parent sa1::sbLink, child sa1::cwaLink, axis 0 0 1
- added joint sa2::j_a_sb: type fixed, parent sa2::aLink, child sa2::sbLink
- added joint sa2::j_sb_ccwa: type continuous, parent sa2::sbLink, child sa2::ccwaLink, axis 0 0 1
- added joint sa2::j_sb_cwa: type continuous, parent sa2::sbLink, child sa2::cwaLink, axis 0 0 1
- added joint sa3::j_a_sb: type fixed, parent sa3::aLink, child sa3::sbLink
- added joint sa3::j_sb_ccwa: type continuous, parent sa3::sbLink, child sa3::ccwaLink, axis 0 0 1
- added joint sa3::j_sb_cwa: type continuous, parent sa3::sbLink, child sa3::cwaLink, axis 0 0 1
- added joint wa2::j_a_wb: type fixed, parent wa2::aLink, child wa2::wbLink
- added joint wa2::j_wb_fw: type continuous, parent wa2::wbLink, child wa2::fwLink, axis 0 0 1
- added joint wa2::j_wb_rw: type continuous, parent wa2::wbLink, child wa2::rwLink, axis 0 0 1
- added joint wa3::j_a_wb: type fixed, parent wa3::aLink, child wa3::wbLink
- added joint wa3::j_wb_fw: type continuous, parent wa3::wbLink, child wa3::fwLink, axis 0 0 1
- added joint wa3::j_wb_rw: type continuous, parent wa3::wbLink, child wa3::rwLink, axis 0 0 1
- joint j_b_l1: origin xyz=0 0 0 rpy=0.083 0 0.075 -> xyz=0.0035 0.024 0.0473 rpy=0 0 0; parent b::bLink -> base_link
- joint j_b_l2: origin xyz=-2.0944 0 0 rpy=0.083 0.065 -0.0375 -> xyz=0.083 0.065 -0.0375 rpy=-2.0944 0 0; parent b::bLink -> base_link
- joint j_b_l3: origin xyz=-2.0944 0 0 rpy=0.083 -0.065 -0.0375 -> xyz=0.083 -0.065 -0.0375 rpy=2.0944 0 0; parent b::bLink -> base_link

Commit message: add urdf, compatible with nav2

File: models/rm2/rm2.urdf (robot description, URDF)
Before this commit: robot rm2_sim, 31 links, 30 joints
Links:
- removed link sa1::ccwaLink
- removed link sa1::cwaLink
- removed link sa2::ccwaLink
- removed link sa2::cwaLink
- removed link sa3::ccwaLink
- removed link sa3::cwaLink
- removed link wa2::fwLink
- removed link wa2::rwLink
- removed link wa3::fwLink
- removed link wa3::rwLink
- added link lidar
Joints:
- removed joint sa1::j_sb_ccwa
- removed joint sa1::j_sb_cwa
- removed joint sa2::j_sb_ccwa
- removed joint sa2::j_sb_cwa
- removed joint sa3::j_sb_ccwa
- removed joint sa3::j_sb_cwa
- removed joint wa2::j_wb_fw
- removed joint wa2::j_wb_rw
- removed joint wa3::j_wb_fw
- removed joint wa3::j_wb_rw
- added joint j_lidar_b: type fixed, parent base_link, child lidar, origin xyz=0.0 0 0.25 rpy=0 0 0
- joint l1::j_l_m: origin (none) -> xyz=0 0 0 rpy=0 0 0
- joint l1::j_m_f: origin (none) -> xyz=0.0153 0.019 0.0135 rpy=0 0 0
- joint l2::j_l_m: origin (none) -> xyz=0 0 0 rpy=0 0 0
- joint l2::j_m_f: origin (none) -> xyz=0.0153 0.019 0.0135 rpy=0 0 0
- joint l3::j_l_m: origin (none) -> xyz=0 0 0 rpy=0 0 0
- joint l3::j_m_f: origin (none) -> xyz=0.0153 0.019 0.0135 rpy=0 0 0
- joint sa1::j_a_sb: origin (none) -> xyz=0 0 0 rpy=0 0 0
- joint sa2::j_a_sb: origin (none) -> xyz=0 0 0 rpy=0 0 0
- joint sa3::j_a_sb: origin (none) -> xyz=0 0 0 rpy=0 0 0
- joint wa2::j_a_wb: origin (none) -> xyz=0 0 0.0025 rpy=0 1.5708 0
- joint wa3::j_a_wb: origin (none) -> xyz=0 0 0.0025 rpy=0 1.5708 0

Commit message: solved wheels pose pub, edgar cave

File: models/rm2/rm2.urdf (robot description, URDF)
Before this commit: robot rm2_sim, 22 links, 21 joints
Links:
- added link sa1::ccwaLink
- added link sa1::cwaLink
- added link sa2::ccwaLink
- added link sa2::cwaLink
- added link sa3::ccwaLink
- added link sa3::cwaLink
- added link wa2::fwLink
- added link wa2::rwLink
- added link wa3::fwLink
- added link wa3::rwLink
Joints:
- added joint sa1::j_sb_ccwa: type continuous, parent sa1::sbLink, child sa1::ccwaLink, origin xyz=-0.010 0 0.0025 rpy=0 -1.5708 0, axis 0 0 1
- added joint sa1::j_sb_cwa: type continuous, parent sa1::sbLink, child sa1::cwaLink, origin xyz=0.010 0 0.0025 rpy=0 1.5708 0, axis 0 0 1
- added joint sa2::j_sb_ccwa: type continuous, parent sa2::sbLink, child sa2::ccwaLink, origin xyz=-0.010 0 0.0025 rpy=0 -1.5708 0, axis 0 0 1
- added joint sa2::j_sb_cwa: type continuous, parent sa2::sbLink, child sa2::cwaLink, origin xyz=0.010 0 0.0025 rpy=0 1.5708 0, axis 0 0 1
- added joint sa3::j_sb_ccwa: type continuous, parent sa3::sbLink, child sa3::ccwaLink, origin xyz=-0.010 0 0.0025 rpy=0 1.5708 0, axis 0 0 1
- added joint sa3::j_sb_cwa: type continuous, parent sa3::sbLink, child sa3::cwaLink, origin xyz=0.010 0 0.0025 rpy=0 1.5708 0, axis 0 0 1
- added joint wa2::j_wb_fw: type continuous, parent wa2::wbLink, child wa2::fwLink, origin xyz=0.009 0 0.07425 rpy=1.5708 0 0, axis 0 0 1
- added joint wa2::j_wb_rw: type continuous, parent wa2::wbLink, child wa2::rwLink, origin xyz=0.009 0 -0.07425 rpy=1.5708 0 0, axis 0 0 1
- added joint wa3::j_wb_fw: type continuous, parent wa3::wbLink, child wa3::fwLink, origin xyz=0.009 0 0.07425 rpy=1.5708 0 0, axis 0 0 1
- added joint wa3::j_wb_rw: type continuous, parent wa3::wbLink, child wa3::rwLink, origin xyz=0.009 0 -0.07425 rpy=1.5708 0 0, axis 0 0 1
- joint j_b_l1: origin xyz=0.0035 0.024 0.0473 rpy=0 0 0 -> xyz=0.083 0 0.075 rpy=0 0 0

Commit message: wheels corrected and urdf trial

File: models/rm2/rm2.urdf (robot description, URDF)
Before this commit: robot rm2_sim, 32 links, 31 joints
Links:
- removed link sa1::ccwaLink
- removed link sa1::cwaLink
- removed link sa2::ccwaLink
- removed link sa2::cwaLink
- removed link sa3::ccwaLink
- removed link sa3::cwaLink
- added link sa1::ccwsLink
- added link sa1::cwsLink
- added link sa2::ccwsLink
- added link sa2::cwsLink
- added link sa3::ccwsLink
- added link sa3::cwsLink
- link base_link: geometry visual mesh filename=rm2_simulation:model://models/rm2/rm2_body/meshes/body_stru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
Joints:
- removed joint sa1::j_sb_ccwa
- removed joint sa1::j_sb_cwa
- removed joint sa2::j_sb_ccwa
- removed joint sa2::j_sb_cwa
- removed joint sa3::j_sb_ccwa
- removed joint sa3::j_sb_cwa
- added joint sa1::j_sb_ccws: type continuous, parent sa1::sbLink, child sa1::ccwsLink, origin xyz=-0.0145 -0.024 0.0132 rpy=0 -1.5708 0, axis 0 0 1
- added joint sa1::j_sb_cws: type continuous, parent sa1::sbLink, child sa1::cwsLink, origin xyz=0.0055 -0.024 0.0132 rpy=0 1.5708 0, axis 0 0 1
- added joint sa2::j_sb_ccws: type continuous, parent sa2::sbLink, child sa2::ccwsLink, origin xyz=-0.0145 -0.024 0.0132 rpy=0 -1.5708 0, axis 0 0 1
- added joint sa2::j_sb_cws: type continuous, parent sa2::sbLink, child sa2::cwsLink, origin xyz=0.0055 -0.024 0.0132 rpy=0 1.5708 0, axis 0 0 1
- added joint sa3::j_sb_ccws: type continuous, parent sa3::sbLink, child sa3::ccwsLink, origin xyz=-0.0145 -0.024 0.0132 rpy=0 -1.5708 0, axis 0 0 1
- added joint sa3::j_sb_cws: type continuous, parent sa3::sbLink, child sa3::cwsLink, origin xyz=0.0055 -0.024 0.0132 rpy=0 1.5708 0, axis 0 0 1
- joint j_l1_sa1: origin xyz=0.0035 0.024 0.0473 rpy=0 0 0 -> xyz=-0.0127 0.005 0.092 rpy=0 0 0
- joint j_l2_sa2: origin xyz=0.0035 0.024 0.0473 rpy=0 0 0 -> xyz=-0.0127 0.005 0.092 rpy=0 0 0
- joint j_l2_wa2: origin xyz=0.0035 0.024 0.0473 rpy=0 0 0 -> xyz=-0.0127 0.005 0.092 rpy=0 0 0
- joint j_l3_sa3: origin xyz=0.0035 0.024 0.0473 rpy=0 0 0 -> xyz=-0.0127 0.005 0.092 rpy=0 0 0
- joint j_l3_wa3: origin xyz=0.0035 0.024 0.0473 rpy=0 0 0 -> xyz=-0.0127 0.005 0.092 rpy=0 0 0
- joint j_lidar_b: origin xyz=0.0 0 0.25 rpy=0 0 0 -> xyz=0 0 0.25 rpy=0 0 0
- joint l1::j_m_f: origin xyz=0.0153 0.019 0.0135 rpy=0 0 0 -> xyz=-0.0669 0.019 0.024 rpy=0 0 0
- joint l2::j_l_m: origin xyz=0 0 0 rpy=0 0 0 -> xyz=0 0 0 rpy=-0.523599 0 0
- joint l2::j_m_f: origin xyz=0.0153 0.019 0.0135 rpy=0 0 0 -> xyz=-0.0669 0.019 0.024 rpy=0 0 0
- joint l3::j_l_m: origin xyz=0 0 0 rpy=0 0 0 -> xyz=0 0 0 rpy=0.523599 0 0
- joint l3::j_m_f: origin xyz=0.0153 0.019 0.0135 rpy=0 0 0 -> xyz=-0.0669 0.019 0.024 rpy=0 0 0
- joint wa2::j_a_wb: origin xyz=0 0 0.0025 rpy=0 1.5708 0 -> xyz=-0.0045 -0.024 0.0132 rpy=0 -0.523599 1.5708
- joint wa2::j_wb_fw: origin xyz=0.009 0 0.07425 rpy=1.5708 0 0 -> xyz=0.009 0 0.040 rpy=1.5708 0 0
- joint wa2::j_wb_rw: origin xyz=0.009 0 -0.07425 rpy=1.5708 0 0 -> xyz=0.009 0 -0.040 rpy=1.5708 0 0
- joint wa3::j_a_wb: origin xyz=0 0 0.0025 rpy=0 1.5708 0 -> xyz=-0.0045 -0.024 0.0132 rpy=0 -0.523599 1.5708
- joint wa3::j_wb_fw: origin xyz=0.009 0 0.07425 rpy=1.5708 0 0 -> xyz=0.009 0 0.040 rpy=1.5708 0 0
- joint wa3::j_wb_rw: origin xyz=0.009 0 -0.07425 rpy=1.5708 0 0 -> xyz=0.009 0 -0.040 rpy=1.5708 0 0
