Commit message: attachabke link working

File: urdf/sensors.xacro (robot description, xacro)
@@ -13,9 +13,9 @@
           izz="0.0000000001" />
       </inertial>
-      <collision name="lidar_collision">
+      <!-- <collision name="lidar_collision">
         <geometry>
           <box size="0.02505 0.09 0.025" />
         </geometry>
-      </collision>
+      </collision> -->
     </link>
     <joint name="joint_${name}" type="fixed">
@@ -35,23 +35,9 @@
           izz="0.0000000001" />
       </inertial>
-      <collision name="d435_camera_collision">
+      <!-- <collision name="d435_camera_collision">
         <geometry>
           <box size="0.02505 0.09 0.025" />
         </geometry>
-        <surface>
-          <contact>
-            <ode>
-              <kp>1e+13</kp>
-              <kd>1</kd>
-            </ode>
-          </contact>
-          <friction>
-            <ode>
-              <mu2>1</mu2>
-              <fdir1>0 0 0</fdir1>
-            </ode>
-          </friction>
-        </surface>
-      </collision>
+      </collision> -->
       <visual name="d435_camera_visual">
         <geometry>
