Commit message: urdf finish diff drive working

File: urdf/rm2.urdf.xacro (robot description, xacro)
@@ -1,23 +1,99 @@
 <?xml version="1.0"?>
 <robot name="rm2_sim" xmlns:xacro="http://www.ros.org/wiki/xacro">
-<!-- <xacro:include filename="$(find robot_sim)/urdf/p3/robot.gazebo" /> -->
-<link name="base_link">
+  <xacro:include filename="$(find rm2_simulation)/urdf/rm2_leg.xacro" />
+  <xacro:include filename="$(find rm2_simulation)/urdf/rm2_screw_actuator.xacro" />
+  <xacro:include filename="$(find rm2_simulation)/urdf/rm2_wheel_actuator.xacro" />
+  <xacro:include filename="$(find rm2_simulation)/urdf/rm2.gazebo" />
+  <link name="base_link">
     <pose>0 0 0 0 0 0</pose>
     <inertial>
-        <mass value="1.114" />
-        <origin rpy="0 0 0" xyz="0 0 0.0" />
-        <inertia ixx="0.00773" ixy="0" ixz="0" iyy="0.00937" iyz="0"
-          izz="0.00938" />
-      </inertial>
+      <mass value="1.114" />
+      <inertia ixx="0.00773" ixy="0" ixz="0" iyy="0.00937" iyz="0"
+        izz="0.00938" />
+    </inertial>
     <collision name='collision_base'>
       <geometry>
-            <mesh filename="file://$(find rm2_simulation)/urdf/meshes/body_collision.stl" scale="0.001 0.001 0.001"/>
+        <mesh filename="file://$(find rm2_simulation)/urdf/meshes/body_collision.stl"
+          scale="0.001 0.001 0.001" />
       </geometry>
     </collision>
     <visual name='visual_base'>
       <geometry>
-        <mesh filename="file://$(find rm2_simulation)/urdf/meshes/body_structure_blue.dae"/>
+        <mesh filename="file://$(find rm2_simulation)/urdf/meshes/body_structure_blue.dae" />
       </geometry>
     </visual>
   </link>
-  </robot>
+  <!-- =================================================================================== -->
+  <!-- |                                          LEGS                                   | -->
+  <!-- =================================================================================== -->
+  <!-- JOINT BODY - SIMPLE LEG 1 -->
+  <joint name="j_b_l1" type="fixed">
+    <origin xyz="0.083 0 0.075" rpy="0 0 0" />
+    <parent link="base_link" />
+    <child link="l1_lLink" />
+  </joint>
+  <!-- INCLUDE SIMPLE LEG 1 -->
+  <xacro:simple_leg name="l1" origin_xyz="-0.0822 0 0.0105" origin_rpy="0 0 0" />
+  <!-- JOINT BODY - SIMPLE LEG 2 (LEFT)-->
+  <joint name="j_b_l2" type="fixed">
+    <origin xyz="0.083 0.065 -0.0375" rpy="-2.0944 0 0" />
+    <parent link="base_link" />
+    <child link="l2_lLink" />
+  </joint>
+  <!-- INCLUDE SIMPLE LEG 2 (LEFT)-->
+  <xacro:simple_leg name="l2" origin_xyz="-0.0822 0 0.0105" origin_rpy="-0.523599 0 0" />
+  <!-- JOINT BODY - SIMPLE LEG 3 (RIGHT)-->
+  <joint name="j_b_l3" type="fixed">
+    <origin xyz="0.083 -0.065 -0.0375" rpy="2.0944 0 0" />
+    <parent link="base_link" />
+    <child link="l3_lLink" />
+  </joint>
+  <!-- INCLUDE SIMPLE LEG 3 (RIGHT)-->
+  <xacro:simple_leg name="l3" origin_xyz="-0.0822 0 0.0105" origin_rpy="0.523599 0 0" />
+  <!-- =================================================================================== -->
+  <!-- |                                      ACTUATORS                                  | -->
+  <!-- =================================================================================== -->
+  <!-- INCLUDE SCREW ACTUATOR 1 -->
+  <xacro:screw_actuator name="sa1" origin_xyz="-0.0045 -0.024 0.0107" origin_rpy="0 0 0" />
+  <!-- JOINT SIMPLE LEG 1 - SCREW ACTUATOR -->
+  <joint name="j_l1_sa1" type="fixed">
+    <origin xyz="-0.0127 0.005 0.092" rpy="0 0 0" />
+    <parent link="l1_fLink" />
+    <child link="sa1_aLink" />
+  </joint>
+  <!-- INCLUDE SCREW ACTUATOR 2 -->
+  <xacro:screw_actuator name="sa2" origin_xyz="-0.0045 -0.024 0.0107" origin_rpy="0 0 0" />
+  <!-- JOINT SIMPLE LEG 2 - SCREW ACTUATOR -->
+  <joint name="j_l1_sa2" type="fixed">
+    <origin xyz="-0.0127 0.005 0.092" rpy="0 0 0" />
+    <parent link="l2_fLink" />
+    <child link="sa2_aLink" />
+  </joint>
+  <!-- INCLUDE SCREW ACTUATOR 3 -->
+  <xacro:screw_actuator name="sa3" origin_xyz="-0.0045 -0.024 0.0107" origin_rpy="0 0 3.14159" />
+  <!-- JOINT SIMPLE LEG 3 - SCREW ACTUATOR -->
+  <joint name="j_l1_sa3" type="fixed">
+    <origin xyz="-0.0127 0.005 0.092" rpy="0 0 0" />
+    <parent link="l3_fLink" />
+    <child link="sa3_aLink" />
+  </joint>
+  <!-- =================================================================================== -->
+  <!-- |                                          WHEELS                                 | -->
+  <!-- =================================================================================== -->
+  <!-- INCLUDE WHEELS ACTUATOR 2 (LEFT) -->
+  <xacro:wheel_actuator name="wa2" origin_xyz="-0.0045 -0.024 0.0107" origin_rpy="0 1.5708 0" />
+  <!-- JOINT SIMPLE LEG 2 - WHEELS ACTUATOR 2 (LEFT) -->
+  <joint name="j_l2_wa2" type="fixed">
+    <origin xyz="-0.0127 0.005 0.092" rpy="0 0 0" />
+    <parent link="l2_fLink" />
+    <child link="wa2_aLink" />
+  </joint>
+  <!-- INCLUDE WHEELS ACTUATOR 3 (LEFT) -->
+  <xacro:wheel_actuator name="wa3" origin_xyz="-0.0045 -0.024 0.0107" origin_rpy="0 1.5708 0" />
+  <!-- JOINT SIMPLE LEG 3 - WHEELS ACTUATOR 3 (LEFT) -->
+  <joint name="j_l3_wa3" type="fixed">
+    <origin xyz="-0.0127 0.005 0.092" rpy="0 0 0" />
+    <parent link="l3_fLink" />
+    <child link="wa3_aLink" />
+  </joint>
+</robot>

Commit message: urdf working, sensors OK

File: urdf/rm2.urdf.xacro (robot description, xacro)
@@ -2,7 +2,12 @@
 <robot name="rm2_sim" xmlns:xacro="http://www.ros.org/wiki/xacro">
   <xacro:include filename="$(find rm2_simulation)/urdf/rm2_leg.xacro" />
-  <xacro:include filename="$(find rm2_simulation)/urdf/rm2_screw_actuator.xacro" />
-  <xacro:include filename="$(find rm2_simulation)/urdf/rm2_wheel_actuator.xacro" />
-  <xacro:include filename="$(find rm2_simulation)/urdf/rm2.gazebo" />
+  <xacro:include
+    filename="$(find rm2_simulation)/urdf/rm2_screw_actuator.xacro" />
+  <xacro:include
+    filename="$(find rm2_simulation)/urdf/rm2_wheel_actuator.xacro" />
+  <xacro:include
+    filename="$(find rm2_simulation)/urdf/rm2.gazebo" />
+  <xacro:include
+    filename="$(find rm2_simulation)/urdf/sensors.xacro" />
   <link name="base_link">
     <pose>0 0 0 0 0 0</pose>
@@ -28,5 +33,6 @@
   <!-- =================================================================================== -->
   <!-- JOINT BODY - SIMPLE LEG 1 -->
-  <joint name="j_b_l1" type="fixed">
+  <joint
+    name="j_b_l1" type="fixed">
     <origin xyz="0.083 0 0.075" rpy="0 0 0" />
     <parent link="base_link" />
@@ -34,5 +40,6 @@
   </joint>
   <!-- INCLUDE SIMPLE LEG 1 -->
-  <xacro:simple_leg name="l1" origin_xyz="-0.0822 0 0.0105" origin_rpy="0 0 0" />
+  <xacro:simple_leg name="l1" origin_xyz="-0.0822 0 0.0105"
+    origin_rpy="0 0 0" />
   <!-- JOINT BODY - SIMPLE LEG 2 (LEFT)-->
   <joint name="j_b_l2" type="fixed">
@@ -42,5 +49,6 @@
   </joint>
   <!-- INCLUDE SIMPLE LEG 2 (LEFT)-->
-  <xacro:simple_leg name="l2" origin_xyz="-0.0822 0 0.0105" origin_rpy="-0.523599 0 0" />
+  <xacro:simple_leg name="l2" origin_xyz="-0.0822 0 0.0105"
+    origin_rpy="-0.523599 0 0" />
   <!-- JOINT BODY - SIMPLE LEG 3 (RIGHT)-->
   <joint name="j_b_l3" type="fixed">
@@ -50,10 +58,12 @@
   </joint>
   <!-- INCLUDE SIMPLE LEG 3 (RIGHT)-->
-  <xacro:simple_leg name="l3" origin_xyz="-0.0822 0 0.0105" origin_rpy="0.523599 0 0" />
+  <xacro:simple_leg name="l3" origin_xyz="-0.0822 0 0.0105"
+    origin_rpy="0.523599 0 0" />
   <!-- =================================================================================== -->
   <!-- |                                      ACTUATORS                                  | -->
   <!-- =================================================================================== -->
   <!-- INCLUDE SCREW ACTUATOR 1 -->
-  <xacro:screw_actuator name="sa1" origin_xyz="-0.0045 -0.024 0.0107" origin_rpy="0 0 0" />
+  <xacro:screw_actuator name="sa1" origin_xyz="-0.0045 -0.024 0.0107"
+    origin_rpy="0 0 0" />
   <!-- JOINT SIMPLE LEG 1 - SCREW ACTUATOR -->
   <joint name="j_l1_sa1" type="fixed">
@@ -63,5 +73,6 @@
   </joint>
   <!-- INCLUDE SCREW ACTUATOR 2 -->
-  <xacro:screw_actuator name="sa2" origin_xyz="-0.0045 -0.024 0.0107" origin_rpy="0 0 0" />
+  <xacro:screw_actuator name="sa2"
+    origin_xyz="-0.0045 -0.024 0.0107" origin_rpy="0 0 0" />
   <!-- JOINT SIMPLE LEG 2 - SCREW ACTUATOR -->
   <joint name="j_l1_sa2" type="fixed">
@@ -71,7 +82,9 @@
   </joint>
   <!-- INCLUDE SCREW ACTUATOR 3 -->
-  <xacro:screw_actuator name="sa3" origin_xyz="-0.0045 -0.024 0.0107" origin_rpy="0 0 3.14159" />
+  <xacro:screw_actuator name="sa3"
+    origin_xyz="-0.0045 -0.024 0.0107" origin_rpy="0 0 3.14159" />
   <!-- JOINT SIMPLE LEG 3 - SCREW ACTUATOR -->
-  <joint name="j_l1_sa3" type="fixed">
+  <joint name="j_l1_sa3"
+    type="fixed">
     <origin xyz="-0.0127 0.005 0.092" rpy="0 0 0" />
     <parent link="l3_fLink" />
@@ -82,5 +95,6 @@
   <!-- =================================================================================== -->
   <!-- INCLUDE WHEELS ACTUATOR 2 (LEFT) -->
-  <xacro:wheel_actuator name="wa2" origin_xyz="-0.0045 -0.024 0.0107" origin_rpy="0 1.5708 0" />
+  <xacro:wheel_actuator name="wa2"
+    origin_xyz="-0.0045 -0.024 0.0107" origin_rpy="0 1.5708 0" />
   <!-- JOINT SIMPLE LEG 2 - WHEELS ACTUATOR 2 (LEFT) -->
   <joint name="j_l2_wa2" type="fixed">
@@ -90,5 +104,6 @@
   </joint>
   <!-- INCLUDE WHEELS ACTUATOR 3 (LEFT) -->
-  <xacro:wheel_actuator name="wa3" origin_xyz="-0.0045 -0.024 0.0107" origin_rpy="0 1.5708 0" />
+  <xacro:wheel_actuator name="wa3"
+    origin_xyz="-0.0045 -0.024 0.0107" origin_rpy="0 1.5708 0" />
   <!-- JOINT SIMPLE LEG 3 - WHEELS ACTUATOR 3 (LEFT) -->
   <joint name="j_l3_wa3" type="fixed">
@@ -97,3 +112,121 @@
     <child link="wa3_aLink" />
   </joint>
+  <!-- =================================================================================== -->
+  <!-- |                                          SENSORS                                | -->
+  <!-- =================================================================================== -->
+  <!-- INCLUDE IMU-->
+  <gazebo reference="base_link">
+    <sensor name="imu_sensor" type="imu">
+      <always_on>1</always_on>
+      <update_rate>1</update_rate>
+      <visualize>true</visualize>
+      <topic>imu</topic>
+      <imu>
+        <angular_velocity>
+          <x>
+            <noise type="gaussian">
+              <mean>0.0</mean>
+              <stddev>2e-4</stddev>
+              <bias_mean>0.0000075</bias_mean>
+              <bias_stddev>0.0000008</bias_stddev>
+            </noise>
+          </x>
+          <y>
+            <noise type="gaussian">
+              <mean>0.0</mean>
+              <stddev>2e-4</stddev>
+              <bias_mean>0.0000075</bias_mean>
+              <bias_stddev>0.0000008</bias_stddev>
+            </noise>
+          </y>
+          <z>
+            <noise type="gaussian">
+              <mean>0.0</mean>
+              <stddev>2e-4</stddev>
+              <bias_mean>0.0000075</bias_mean>
+              <bias_stddev>0.0000008</bias_stddev>
+            </noise>
+          </z>
+        </angular_velocity>
+        <linear_acceleration>
+          <x>
+            <noise type="gaussian">
+              <mean>0.0</mean>
+              <stddev>1.7e-2</stddev>
+              <bias_mean>0.1</bias_mean>
+              <bias_stddev>0.001</bias_stddev>
+            </noise>
+          </x>
+          <y>
+            <noise type="gaussian">
+              <mean>0.0</mean>
+              <stddev>1.7e-2</stddev>
+              <bias_mean>0.1</bias_mean>
+              <bias_stddev>0.001</bias_stddev>
+            </noise>
+          </y>
+          <z>
+            <noise type="gaussian">
+              <mean>0.0</mean>
+              <stddev>1.7e-2</stddev>
+              <bias_mean>0.1</bias_mean>
+              <bias_stddev>0.001</bias_stddev>
+            </noise>
+          </z>
+        </linear_acceleration>
+      </imu>
+    </sensor>
+  </gazebo>
+  <!-- INCLUDE LASER-->
+  <xacro:laser name="lidar" parent="base_link" />
+  <gazebo reference="lidar">
+    <sensor name="front_lidar" type="gpu_lidar">
+      <topic>/laserscan</topic>
+      <always_on>true</always_on>
+      <visualize>false</visualize>
+      <update_rate>10</update_rate>
+      <always_on>1</always_on>
+      <ray>
+        <scan>
+          <horizontal>
+            <samples>720</samples>
+            <resolution>1</resolution>
+            <min_angle>-1.8326</min_angle>
+            <max_angle>1.8326</max_angle>
+          </horizontal>
+        </scan>
+        <range>
+          <min>0.05</min>
+          <max>20</max>
+          <resolution>0.01</resolution>
+        </range>
+        <noise>
+          <type>gaussian</type>
+          <mean>0</mean>
+          <stddev>0.01</stddev>
+        </noise>
+      </ray>
+    </sensor>
+  </gazebo>
+  <!-- INCLUDE CAMERA-->
+  <xacro:realsense_camera name="d_435_camera" parent="base_link" />
+  <gazebo reference="d_435_camera">
+    <sensor name="rgbd_camera" type="rgbd_camera">
+      <always_on>true</always_on>
+      <update_rate>30</update_rate>
+      <visualize>false</visualize>
+      <topic>/rgbd_camera</topic>
+      <camera>
+        <horizontal_fov>1.05</horizontal_fov>
+        <image>
+          <width>256</width>
+          <height>256</height>
+        </image>
+        <clip>
+          <near>0.1</near>
+          <far>10.0</far>
+        </clip>
+      </camera>
+      </sensor>
+  </gazebo>
 </robot>

File: urdf/rm2_wheel_actuator.xacro (robot description, xacro)
@@ -5,7 +5,7 @@
         <link name="${name}_aLink">
             <inertial>
-                <mass value="0.001" />
-                <inertia ixx="0.00012" ixy="0" ixz="0" iyy="0.00096" iyz="0"
-                    izz="0.00094" />
+                <mass value="0.0" />
+                <inertia ixx="0.0" ixy="0" ixz="0" iyy="0.0" iyz="0"
+                    izz="0.0" />
             </inertial>
         </link>
@@ -33,5 +33,5 @@
         <!-- JOINT ACTUATOR - WHEELS BAR -->
         <joint name="${name}_j_a_wb" type="fixed">
-            <origin rpy="${origin_rpy}" xyz="${origin_xyz}"/>
+            <origin rpy="${origin_rpy}" xyz="${origin_xyz}" />
             <parent link="${name}_aLink" />
             <child link="${name}_wbLink" />
@@ -42,9 +42,9 @@
                 <mass value="0.1" />
                 <inertia ixx="0.064" ixy="0" ixz="0" iyy="0.064" iyz="0"
-                    izz="0.064" />
+                    izz="0.00024" />
             </inertial>
             <collision name='collision_base'>
                 <geometry>
-                    <cylinder length="0.01" radius="0.03" />
+                    <cylinder length="0.08" radius="0.028" />
                 </geometry>
             </collision>
@@ -73,9 +73,9 @@
                 <mass value="0.1" />
                 <inertia ixx="0.064" ixy="0" ixz="0" iyy="0.064" iyz="0"
-                    izz="0.064" />
+                    izz="0.00024" />
             </inertial>
             <collision name='collision_base'>
                 <geometry>
-                    <cylinder length="0.01" radius="0.03" />
+                    <cylinder length="0.08" radius="0.03" />
                 </geometry>
             </collision>

Commit message: add cutting head and coupling disk URDF

File: urdf/rm2.urdf.xacro (robot description, xacro)
@@ -111,4 +111,53 @@
     <parent link="l3_fLink" />
     <child link="wa3_aLink" />
+  </joint>
+  <!-- =================================================================================== -->
+  <!-- |                                     COUPLING DISK                                |-->
+  <!-- =================================================================================== -->
+  <link name="couplingLink">
+    <inertial>
+      <mass value="1.114" />
+      <inertia ixx="0.00773" ixy="0" ixz="0" iyy="0.00937" iyz="0" izz="0.00938" />
+    </inertial>
+    <collision name='collision_coupling'>
+      <geometry>
+        <mesh filename="file://$(find rm2_simulation)/urdf/meshes/coupling_head.dae" />
+      </geometry>
+    </collision>
+    <visual name='visual_'>
+      <geometry>
+        <mesh filename="file://$(find rm2_simulation)/urdf/meshes/coupling_head.dae" />
+      </geometry>
+    </visual>
+  </link>
+  <joint name="j_c_b" type="fixed">
+    <origin xyz="0.10196 0.0 0.0" rpy="0 0 0" />
+    <parent link="base_link" />
+    <child link="couplingLink" />
+  </joint>
+  <!-- =================================================================================== -->
+  <!-- |                                     CUTTING HEAD                                 |-->
+  <!-- =================================================================================== -->
+  <link name="cuttingHeadLink">
+    <inertial>
+      <mass value="0.114" />
+      <inertia ixx="0.00773" ixy="0" ixz="0" iyy="0.00937" iyz="0" izz="0.00938" />
+    </inertial>
+    <collision name='collision_head'>
+      <geometry>
+        <mesh filename="file://$(find rm2_simulation)/urdf/meshes/cutting_head_simple.dae"/>
+      </geometry>
+    </collision>
+    <visual name='visual_head'>
+      <geometry>
+        <mesh filename="file://$(find rm2_simulation)/urdf/meshes/cutting_head_simple.dae" />
+      </geometry>
+    </visual>
+  </link>
+  <joint name="j_ch_c" type="fixed">
+    <origin xyz="0.09315
+    + 0.0 0.0" rpy="0 0 0" />
+    <parent link="couplingLink" />
+    <child link="cuttingHeadLink" />
   </joint>
   <!-- =================================================================================== -->

Commit message: tested OK

File: urdf/rm2.urdf.xacro (robot description, xacro)
@@ -115,5 +115,5 @@
   <!-- |                                     COUPLING DISK                                |-->
   <!-- =================================================================================== -->
-  <link name="couplingLink">
+  <!-- <link name="couplingLink">
     <inertial>
       <mass value="1.114" />
@@ -135,9 +135,9 @@
     <parent link="base_link" />
     <child link="couplingLink" />
-  </joint>
+  </joint> -->
   <!-- =================================================================================== -->
   <!-- |                                     CUTTING HEAD                                 |-->
   <!-- =================================================================================== -->
-  <link name="cuttingHeadLink">
+  <!-- <link name="cuttingHeadLink">
     <inertial>
       <mass value="0.114" />
@@ -160,5 +160,5 @@
     <parent link="couplingLink" />
     <child link="cuttingHeadLink" />
-  </joint>
+  </joint> -->
   <!-- =================================================================================== -->
   <!-- |                                          SENSORS                                | -->

File: urdf/rm2_leg.xacro (robot description, xacro)
@@ -24,5 +24,5 @@
       <collision name='collision_base'>
         <geometry>
-          <mesh filename="file://$(find rm2_simulation)/urdf/meshes/motors.stl"
+          <mesh filename="file://$(find rm2_simulation)/urdf/meshes/motors.dae"
             scale="0.001 0.001 0.001" />
         </geometry>
