Commit message: escenario 3

File: urdf/rm2.urdf.xacro (robot description, xacro)
@@ -13,5 +13,5 @@
     <pose>0 0 0 0 0 0</pose>
     <inertial>
-      <mass value="1.114" />
+      <mass value="0.114" />
       <inertia ixx="0.00773" ixy="0" ixz="0" iyy="0.00937" iyz="0"
         izz="0.00938" />
@@ -115,8 +115,8 @@
   <!-- |                                     COUPLING DISK                                |-->
   <!-- =================================================================================== -->
-  <!-- <link name="couplingLink">
+  <link name="couplingLink">
     <inertial>
-      <mass value="1.114" />
-      <inertia ixx="0.00773" ixy="0" ixz="0" iyy="0.00937" iyz="0" izz="0.00938" />
+      <mass value="0.000000001" />
+      <inertia ixx="0.000000773" ixy="0" ixz="0" iyy="0.0000000937" iyz="0" izz="0.00000000938" />
     </inertial>
     <collision name='collision_coupling'>
@@ -125,5 +125,5 @@
       </geometry>
     </collision>
-    <visual name='visual_'>
+    <visual name='visual_collision'>
       <geometry>
         <mesh filename="file://$(find rm2_simulation)/urdf/meshes/coupling_head.dae" />
@@ -135,12 +135,12 @@
     <parent link="base_link" />
     <child link="couplingLink" />
-  </joint> -->
+  </joint>
   <!-- =================================================================================== -->
   <!-- |                                     CUTTING HEAD                                 |-->
   <!-- =================================================================================== -->
-  <!-- <link name="cuttingHeadLink">
+  <link name="cuttingHeadLink">
     <inertial>
-      <mass value="0.114" />
-      <inertia ixx="0.00773" ixy="0" ixz="0" iyy="0.00937" iyz="0" izz="0.00938" />
+       <mass value="0.000000001" />
+      <inertia ixx="0.000000773" ixy="0" ixz="0" iyy="0.0000000937" iyz="0" izz="0.00000000938" />
     </inertial>
     <collision name='collision_head'>
@@ -156,9 +156,8 @@
   </link>
   <joint name="j_ch_c" type="fixed">
-    <origin xyz="0.09315
-    + 0.0 0.0" rpy="0 0 0" />
+    <origin xyz="0.09315 0.0 0.0" rpy="0 0 0" />
     <parent link="couplingLink" />
     <child link="cuttingHeadLink" />
-  </joint> -->
+  </joint>
   <!-- =================================================================================== -->
   <!-- |                                          SENSORS                                | -->

File: urdf/rm2_leg.xacro (robot description, xacro)
@@ -18,5 +18,5 @@
     <link name="${name}_mLink">
       <inertial>
-        <mass value="0.393" />
+        <mass value="0.003" />
         <inertia ixx="0.00012" ixy="0" ixz="0" iyy="0.00096" iyz="0"
           izz="0.00094" />
@@ -43,5 +43,5 @@
     <link name="${name}_fLink">
       <inertial>
-        <mass value="0.044" />
+        <mass value="0.004" />
         <inertia ixx="0.00007" ixy="0" ixz="0" iyy="0.00012" iyz="0"
           izz="0.00009" />

File: urdf/rm2_screw_actuator.xacro (robot description, xacro)
@@ -18,5 +18,5 @@
         <link name="${name}_sbLink">
             <inertial>
-                <mass value="0.2" />
+                <mass value="0.002" />
                 <inertia ixx="0.064" ixy="0" ixz="0" iyy="0.064" iyz="0"
                     izz="0.00024" />
@@ -49,5 +49,5 @@
         <link name="${name}_cwsLink">
             <inertial>
-                <mass value="0.2" />
+                <mass value="0.002" />
                 <inertia ixx="0.064" ixy="0" ixz="0" iyy="0.064" iyz="0" izz="0.00024" />
             </inertial>
@@ -79,5 +79,5 @@
         <link name="${name}_ccwsLink">
             <inertial>
-                <mass value="0.2" />
+                <mass value="0.002" />
                 <inertia ixx="0.064" ixy="0" ixz="0" iyy="0.064" iyz="0" izz="0.00024" />
             </inertial>

File: urdf/rm2_wheel_actuator.xacro (robot description, xacro)
@@ -5,5 +5,5 @@
         <link name="${name}_aLink">
             <inertial>
-                <mass value="0.0" />
+                <mass value="0.001" />
                 <inertia ixx="0.0" ixy="0" ixz="0" iyy="0.0" iyz="0"
                     izz="0.0" />
@@ -13,5 +13,5 @@
         <link name="${name}_wbLink">
             <inertial>
-                <mass value="0.2" />
+                <mass value="0.002" />
                 <inertia ixx="0.064" ixy="0" ixz="0" iyy="0.064" iyz="0"
                     izz="0.064" />
@@ -40,5 +40,5 @@
         <link name="${name}_fwLink">
             <inertial>
-                <mass value="0.1" />
+                <mass value="0.001" />
                 <inertia ixx="0.064" ixy="0" ixz="0" iyy="0.064" iyz="0"
                     izz="0.00024" />
@@ -71,5 +71,5 @@
         <link name="${name}_rwLink">
             <inertial>
-                <mass value="0.1" />
+                <mass value="0.0001" />
                 <inertia ixx="0.064" ixy="0" ixz="0" iyy="0.064" iyz="0"
                     izz="0.00024" />
